File: esp12.brd (EAGLE design)
At the start: 49.7 x 49.8 mm, 26 parts, among them IC1 117\33

Commit message: gitignore and ADC 5V to 1.8V conversion
Parts:
- added R12: 1k8, resistor:M1206
- added R13: 1k, resistor:M1206
Connections:
- new net ADC: R12.2, R13.1, U$1.ADC
- net GND: now also R13.2
- net N$9: now also R12.1; no longer U$1.ADC
Routing:
- net ADC: track 0.00 -> 18.0 mm, vias 0 -> 1
- net N$9: track 7.08 -> 12.2 mm, vias 0 -> 1
- net GND: track 0.00 -> 4.60 mm, vias 6 -> 10

Commit message: LED for GPIO0 added
Parts:
- added LED1: (no value), led:1206
- added R14: 1k, resistor:M1206
Connections:
- new net N$8: LED1.A, R14.1
- net GND: now also LED1.C
- net GPIO0: now also R14.2
Routing:
- net GPIO0: track 57.9 -> 73.7 mm, vias 2 -> 3
- net GND: track 4.60 -> 9.52 mm
- net N$8: track 0.00 -> 4.32 mm
Changed lines of the file:
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@@
 <attribute name="VALUE" x="5.08" y="47.752" size="1.27" layer="27" font="vector" rot="R270"/>
+</element>
+<element name="LED1" library="led" package="1206" value="" x="40.64" y="46.736" rot="R270"/>
+<element name="R14" library="resistor" package="M1206" value="1k" x="36.322" y="46.736" smashed="yes" rot="R270">
+<attribute name="VALUE" x="33.782" y="48.006" size="1.27" layer="27" rot="R270"/>
 </element>
 </elements>
@@
 <via x="27.432" y="20.32" extent="1-16" drill="0.6"/>
 <via x="13.97" y="20.32" extent="1-16" drill="0.6"/>
+<contactref element="LED1" pad="C"/>
+<wire x1="40.64" y1="45.314" x2="43.18" y2="43.942" width="0.4064" layer="1"/>
+<wire x1="43.18" y1="43.942" x2="43.18" y2="41.91" width="0.4064" layer="1"/>
 </signal>
 <signal name="+3V3">
@@
 <wire x1="29.464" y1="23.5966" x2="29.464" y2="22.8854" width="0.4064" layer="1"/>
 <wire x1="29.464" y1="22.8854" x2="34.5694" y2="17.78" width="0.4064" layer="1"/>
+<contactref element="R14" pad="2"/>
+<wire x1="36.322" y1="45.336" x2="35.176" y2="45.336" width="0.4064" layer="1"/>
+<wire x1="35.176" y1="45.336" x2="34.29" y2="44.45" width="0.4064" layer="1"/>
+<via x="34.29" y="44.45" extent="1-16" drill="0.6"/>
+<wire x1="34.29" y1="44.45" x2="34.29" y2="34.63" width="0.4064" layer="16"/>
+<wire x1="34.29" y1="34.63" x2="33.274" y2="33.782" width="0.4064" layer="16"/>
+<wire x1="33.274" y1="33.782" x2="31.37" y2="33.782" width="0.4064" layer="16"/>
+<wire x1="31.37" y1="33.782" x2="31.03" y2="33.868" width="0.4064" layer="16"/>
 </signal>
 <signal name="GPIO2">
@@
 <wire x1="10.544" y1="47.882" x2="9.906" y2="47.752" width="0.4064" layer="1"/>
 </signal>
+<signal name="N$8">
+<contactref element="LED1" pad="A"/>
+<contactref element="R14" pad="1"/>
+<wire x1="36.322" y1="48.136" x2="40.544" y2="48.136" width="0.4064" layer="1"/>
+<wire x1="40.544" y1="48.136" x2="40.64" y2="48.158" width="0.4064" layer="1"/>
+</signal>
 </signals>
