File: esp12.sch (EAGLE design)
At the start: 30 parts, among them IC1 117\33

Commit message: 100nF because of regulator
Parts:
- C1: value 10uF -> 100nF
Changed lines of the file:
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@@
 <parts>
 <part name="IC1" library="v-reg" deviceset="LD117A?*" device="S" technology="33TR" value="117\33"/>
-<part name="C1" library="resistor" deviceset="C-EU" device="C1206" value="10uF"/>
+<part name="C1" library="resistor" deviceset="C-EU" device="C1206" value="100nF"/>
 <part name="C2" library="resistor" deviceset="C-EU" device="C1206" value="10uF"/>
 <part name="+3V1" library="supply1" deviceset="+3V3" device=""/>
