File: esp12e_3V3.sch (EAGLE design)
At the start: 30 parts, among them CN1 1X4-CLEANBIG, CN2 1X4-CLEANBIG, CN3 1X4-CLEANBIG, IC1 117\33

Commit message: moved 5V header, ftdi and added micro usbfootprint
Parts:
- added CN4: (no value), adafruit:USBMINIB
- JP2: value M02LOCK -> M02PTH; device SparkFun-Connectors:M02LOCK -> SparkFun-Connectors:M02PTH
Connections:
- removed net FRX_ETX: JP1.RXI, JP5.1, U$2.TXD, U$3.TX
- removed net FTX_ERX: JP1.TXO, JP5.2, U$2.RXD, U$3.RX
- new net ERX: JP1.RXI, JP5.2, U$2.RXD, U$3.RX
- new net ETX: JP1.TXO, JP5.1, U$2.TXD, U$3.TX
- net GND: now also CN4.GND
- net VCC: now also CN4.VBUS
Changed lines of the file:
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@@
 <part name="JP7" library="SparkFun-Connectors" deviceset="M07" device=""/>
 <part name="JP9" library="SparkFun-Connectors" deviceset="M07" device=""/>
-<part name="JP2" library="SparkFun-Connectors" deviceset="M02" device="LOCK"/>
 <part name="+3V10" library="supply1" deviceset="+3V3" device=""/>
 <part name="PCB1" library="dp_pcb" deviceset="PCB_DP_SQUARE" device="-5X5"/>
@@
 <part name="CN2" library="adafruit" deviceset="1X4" device="-CLEANBIG"/>
 <part name="CN3" library="adafruit" deviceset="1X4" device="-CLEANBIG"/>
+<part name="CN4" library="adafruit" deviceset="USB" device="MINIB"/>
+<part name="JP2" library="SparkFun-Connectors" deviceset="M02" device="PTH"/>
 </parts>
 <sheets>
@@
 <instance part="JP7" gate="G$1" x="121.92" y="109.22" rot="R180"/>
 <instance part="JP9" gate="G$1" x="134.62" y="109.22" rot="R180"/>
-<instance part="JP2" gate="G$1" x="27.94" y="101.6" rot="R270"/>
 <instance part="+3V10" gate="G$1" x="-27.94" y="43.18" rot="R270"/>
 <instance part="PCB1" gate="G$1" x="10.16" y="132.08"/>
@@
 <instance part="CN2" gate="G$1" x="134.62" y="127"/>
 <instance part="CN3" gate="G$1" x="121.92" y="127"/>
+<instance part="CN4" gate="G$1" x="40.64" y="116.84" rot="R270"/>
+<instance part="JP2" gate="G$1" x="27.94" y="101.6" rot="R270"/>
 </instances>
 <busses>
@@
 <wire x1="17.78" y1="86.36" x2="17.78" y2="91.44" width="0.1524" layer="91"/>
 <wire x1="17.78" y1="91.44" x2="27.94" y2="91.44" width="0.1524" layer="91"/>
-<wire x1="27.94" y1="91.44" x2="27.94" y2="93.98" width="0.1524" layer="91"/>
+<pinref part="CN4" gate="G$1" pin="VBUS"/>
+<wire x1="45.72" y1="106.68" x2="45.72" y2="111.76" width="0.1524" layer="91"/>
+<wire x1="45.72" y1="111.76" x2="27.94" y2="111.76" width="0.1524" layer="91"/>
+<wire x1="27.94" y1="111.76" x2="27.94" y2="93.98" width="0.1524" layer="91"/>
 <pinref part="JP2" gate="G$1" pin="1"/>
-<wire x1="27.94" y1="93.98" x2="27.94" y2="96.52" width="0.1524" layer="91"/>
+<wire x1="27.94" y1="93.98" x2="27.94" y2="91.44" width="0.1524" layer="91"/>
 <junction x="27.94" y="93.98"/>
 </segment>
@@
 <wire x1="30.48" y1="73.66" x2="30.48" y2="78.74" width="0.1524" layer="91"/>
 <wire x1="30.48" y1="96.52" x2="30.48" y2="93.98" width="0.1524" layer="91"/>
+<pinref part="CN4" gate="G$1" pin="GND"/>
+<wire x1="30.48" y1="93.98" x2="30.48" y2="78.74" width="0.1524" layer="91"/>
+<wire x1="35.56" y1="106.68" x2="35.56" y2="96.52" width="0.1524" layer="91"/>
+<wire x1="35.56" y1="96.52" x2="30.48" y2="96.52" width="0.1524" layer="91"/>
 <pinref part="JP2" gate="G$1" pin="2"/>
-<wire x1="30.48" y1="93.98" x2="30.48" y2="78.74" width="0.1524" layer="91"/>
 <junction x="30.48" y="93.98"/>
 </segment>
@@
 </segment>
 </net>
-<net name="FTX_ERX" class="0">
-<segment>
-<wire x1="-12.7" y1="48.26" x2="-33.02" y2="48.26" width="0.1524" layer="91"/>
-<label x="-12.7" y="48.26" size="1.27" layer="95" xref="yes"/>
-<pinref part="JP1" gate="G$1" pin="TXO"/>
-</segment>
+<net name="ERX" class="0">
 <segment>
 <pinref part="U$2" gate="G$1" pin="RXD"/>
@@
 <pinref part="JP5" gate="G$1" pin="2"/>
 </segment>
+<segment>
+<pinref part="JP1" gate="G$1" pin="RXI"/>
+<wire x1="-33.02" y1="45.72" x2="-10.16" y2="45.72" width="0.1524" layer="91"/>
+<label x="-10.16" y="45.72" size="1.016" layer="95" xref="yes"/>
+</segment>
 </net>
 <net name="N$3" class="0">
@@
 </segment>
 </net>
-<net name="FRX_ETX" class="0">
-<segment>
-<pinref part="JP1" gate="G$1" pin="RXI"/>
-<wire x1="-33.02" y1="45.72" x2="-12.7" y2="45.72" width="0.1524" layer="91"/>
-<label x="-12.7" y="45.72" size="1.27" layer="95" xref="yes"/>
-</segment>
+<net name="ETX" class="0">
 <segment>
 <wire x1="91.44" y1="48.26" x2="88.9" y2="48.26" width="0.1524" layer="91"/>
@@
 <label x="99.06" y="106.68" size="1.27" layer="95" xref="yes"/>
 </segment>
-</net>
+<segment>
+<pinref part="JP1" gate="G$1" pin="TXO"/>
+<wire x1="-33.02" y1="48.26" x2="-10.16" y2="48.26" width="0.1524" layer="91"/>
+<label x="-10.16" y="48.26" size="1.016" layer="95" xref="yes"/>
+</segment>
+</net>

Commit message: moved stuff
Parts:
- removed CN4: (no value), adafruit:USBMINIB
- added JP3: USB_MICROB_PLUGCONN-11752, SparkFun-Connectors:USB_MICROB_PLUGCONN-11752
Connections:
- net GND: now also JP3.GND; no longer CN4.GND
- net VCC: now also JP3.VCC; no longer CN4.VBUS
Changed lines of the file:
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@@
 <part name="CN2" library="adafruit" deviceset="1X4" device="-CLEANBIG"/>
 <part name="CN3" library="adafruit" deviceset="1X4" device="-CLEANBIG"/>
-<part name="CN4" library="adafruit" deviceset="USB" device="MINIB"/>
 <part name="JP2" library="SparkFun-Connectors" deviceset="M02" device="PTH"/>
+<part name="JP3" library="SparkFun-Connectors" deviceset="USB_MICROB_PLUG" device="CONN-11752"/>
+<part name="GND6" library="supply1" deviceset="GND" device=""/>
 </parts>
 <sheets>
@@
 <instance part="CN2" gate="G$1" x="134.62" y="127"/>
 <instance part="CN3" gate="G$1" x="121.92" y="127"/>
-<instance part="CN4" gate="G$1" x="40.64" y="116.84" rot="R270"/>
 <instance part="JP2" gate="G$1" x="27.94" y="101.6" rot="R270"/>
+<instance part="JP3" gate="G$1" x="10.16" y="114.3" rot="R90"/>
+<instance part="GND6" gate="1" x="15.24" y="104.14"/>
 </instances>
 <busses>
@@
 <wire x1="17.78" y1="86.36" x2="17.78" y2="91.44" width="0.1524" layer="91"/>
 <wire x1="17.78" y1="91.44" x2="27.94" y2="91.44" width="0.1524" layer="91"/>
-<pinref part="CN4" gate="G$1" pin="VBUS"/>
-<wire x1="45.72" y1="106.68" x2="45.72" y2="111.76" width="0.1524" layer="91"/>
-<wire x1="45.72" y1="111.76" x2="27.94" y2="111.76" width="0.1524" layer="91"/>
 <wire x1="27.94" y1="111.76" x2="27.94" y2="93.98" width="0.1524" layer="91"/>
 <pinref part="JP2" gate="G$1" pin="1"/>
 <wire x1="27.94" y1="93.98" x2="27.94" y2="91.44" width="0.1524" layer="91"/>
 <junction x="27.94" y="93.98"/>
+<pinref part="JP3" gate="G$1" pin="VCC"/>
+<wire x1="5.08" y1="106.68" x2="5.08" y2="111.76" width="0.1524" layer="91"/>
+<wire x1="5.08" y1="111.76" x2="27.94" y2="111.76" width="0.1524" layer="91"/>
 </segment>
 </net>
@@
 <wire x1="30.48" y1="73.66" x2="30.48" y2="78.74" width="0.1524" layer="91"/>
 <wire x1="30.48" y1="96.52" x2="30.48" y2="93.98" width="0.1524" layer="91"/>
-<pinref part="CN4" gate="G$1" pin="GND"/>
 <wire x1="30.48" y1="93.98" x2="30.48" y2="78.74" width="0.1524" layer="91"/>
-<wire x1="35.56" y1="106.68" x2="35.56" y2="96.52" width="0.1524" layer="91"/>
-<wire x1="35.56" y1="96.52" x2="30.48" y2="96.52" width="0.1524" layer="91"/>
 <pinref part="JP2" gate="G$1" pin="2"/>
 <junction x="30.48" y="93.98"/>
@@
 <wire x1="53.34" y1="73.66" x2="53.34" y2="78.74" width="0.1524" layer="91"/>
 </segment>
+<segment>
+<pinref part="JP3" gate="G$1" pin="GND"/>
+<pinref part="GND6" gate="1" pin="GND"/>
+</segment>
 </net>

Commit message: removed "antenna" - wire on pcb and pulled usb
Changed lines of the file:
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@@
 <pinref part="U$3" gate="G$1" pin="RESET"/>
 <pinref part="JP4" gate="G$1" pin="7"/>
+<label x="50.8" y="53.34" size="1.778" layer="95"/>
 </segment>
 <segment>

Commit message: kitnic.it stuff
Parts:
- removed JP2: M02PTH, SparkFun-Connectors:M02PTH
- added JP6: (no value), pinhead:PINHD-1X3
- R12: value 1k8 -> 39k
- R13: value 1k -> 10k
Connections:
- net +3V3: now also JP6.3
- net GND: now also JP6.2; no longer JP2.2
- net VCC: now also JP6.1; no longer JP2.1
Changed lines of the file:
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@@
 <part name="GND11" library="supply1" deviceset="GND" device=""/>
 <part name="R11" library="resistor" deviceset="R-EU_" device="M1206" value="10k"/>
-<part name="R12" library="resistor" deviceset="R-EU_" device="M1206" value="1k8"/>
-<part name="R13" library="resistor" deviceset="R-EU_" device="M1206" value="1k"/>
+<part name="R12" library="resistor" deviceset="R-EU_" device="M1206" value="39k"/>
+<part name="R13" library="resistor" deviceset="R-EU_" device="M1206" value="10k"/>
 <part name="GND14" library="supply1" deviceset="GND" device=""/>
 <part name="LED1" library="led" deviceset="LED" device="SMT1206"/>
@@
 <part name="CN2" library="adafruit" deviceset="1X4" device="-CLEANBIG"/>
 <part name="CN3" library="adafruit" deviceset="1X4" device="-CLEANBIG"/>
-<part name="JP2" library="SparkFun-Connectors" deviceset="M02" device="PTH"/>
 <part name="JP3" library="SparkFun-Connectors" deviceset="USB_MICROB_PLUG" device="CONN-11752"/>
 <part name="GND6" library="supply1" deviceset="GND" device=""/>
+<part name="JP6" library="pinhead" deviceset="PINHD-1X3" device=""/>
 </parts>
 <sheets>
@@
 <instance part="CN2" gate="G$1" x="134.62" y="127"/>
 <instance part="CN3" gate="G$1" x="121.92" y="127"/>
-<instance part="JP2" gate="G$1" x="27.94" y="101.6" rot="R270"/>
 <instance part="JP3" gate="G$1" x="10.16" y="114.3" rot="R90"/>
 <instance part="GND6" gate="1" x="15.24" y="104.14"/>
+<instance part="JP6" gate="A" x="30.48" y="109.22" rot="R90"/>
 </instances>
 <busses>
@@
 <wire x1="17.78" y1="86.36" x2="17.78" y2="91.44" width="0.1524" layer="91"/>
 <wire x1="17.78" y1="91.44" x2="27.94" y2="91.44" width="0.1524" layer="91"/>
-<wire x1="27.94" y1="111.76" x2="27.94" y2="93.98" width="0.1524" layer="91"/>
-<pinref part="JP2" gate="G$1" pin="1"/>
-<wire x1="27.94" y1="93.98" x2="27.94" y2="91.44" width="0.1524" layer="91"/>
-<junction x="27.94" y="93.98"/>
+<wire x1="27.94" y1="111.76" x2="27.94" y2="106.68" width="0.1524" layer="91"/>
+<wire x1="27.94" y1="106.68" x2="27.94" y2="91.44" width="0.1524" layer="91"/>
 <pinref part="JP3" gate="G$1" pin="VCC"/>
 <wire x1="5.08" y1="106.68" x2="5.08" y2="111.76" width="0.1524" layer="91"/>
 <wire x1="5.08" y1="111.76" x2="27.94" y2="111.76" width="0.1524" layer="91"/>
+<pinref part="JP6" gate="A" pin="1"/>
+<junction x="27.94" y="106.68"/>
 </segment>
 </net>
@@
 <wire x1="30.48" y1="96.52" x2="30.48" y2="93.98" width="0.1524" layer="91"/>
 <wire x1="30.48" y1="93.98" x2="30.48" y2="78.74" width="0.1524" layer="91"/>
-<pinref part="JP2" gate="G$1" pin="2"/>
 <junction x="30.48" y="93.98"/>
+<pinref part="JP6" gate="A" pin="2"/>
+<wire x1="30.48" y1="106.68" x2="30.48" y2="93.98" width="0.1524" layer="91"/>
 </segment>
 <segment>
@@
 <pinref part="+3V1" gate="G$1" pin="+3V3"/>
 <wire x1="45.72" y1="91.44" x2="45.72" y2="86.36" width="0.1524" layer="91"/>
-<wire x1="45.72" y1="86.36" x2="38.1" y2="86.36" width="0.1524" layer="91"/>
-</segment>
-<segment>
+<wire x1="45.72" y1="86.36" x2="40.64" y2="86.36" width="0.1524" layer="91"/>
+<pinref part="JP6" gate="A" pin="3"/>
+<wire x1="40.64" y1="86.36" x2="38.1" y2="86.36" width="0.1524" layer="91"/>
+<wire x1="33.02" y1="106.68" x2="40.64" y2="106.68" width="0.1524" layer="91"/>
+<wire x1="40.64" y1="106.68" x2="40.64" y2="86.36" width="0.1524" layer="91"/>
+</segment>
+<segment>
